Commit message: removed front wheel motors. Fixed issue in kinematics.

File: racecar_description/urdf/base.xacro (robot description, xacro)
@@ -53,14 +53,14 @@
         </xacro:racecar_hinge>
         <!-- Racecar wheel macros -->
-        <xacro:racecar_wheel wheel_prefix="front_left" namespace="${namespace}" parent="left_hinge_link">
+        <xacro:racecar_wheel wheel_prefix="front_left" namespace="${namespace}" parent="left_hinge_link" is_motor="false">
             <origin xyz="0 ${wheel_length/2} 0" rpy="0 0 0" />
         </xacro:racecar_wheel>
-        <xacro:racecar_wheel wheel_prefix="front_right" namespace="${namespace}" parent="right_hinge_link">
+        <xacro:racecar_wheel wheel_prefix="front_right" namespace="${namespace}" parent="right_hinge_link" is_motor="false">
             <origin xyz="0 ${-wheel_length/2} 0" rpy="0 0 0" />
         </xacro:racecar_wheel>
-        <xacro:racecar_wheel wheel_prefix="rear_left" namespace="${namespace}" parent="base_link">
+        <xacro:racecar_wheel wheel_prefix="rear_left" namespace="${namespace}" parent="base_link" is_motor="true">
             <origin xyz="0 ${track/2} 0" rpy="0 0 0" />
         </xacro:racecar_wheel>
-        <xacro:racecar_wheel wheel_prefix="rear_right" namespace="${namespace}" parent="base_link">
+        <xacro:racecar_wheel wheel_prefix="rear_right" namespace="${namespace}" parent="base_link" is_motor="true">
             <origin xyz="0 ${-track/2} 0" rpy="0 0 0" />
         </xacro:racecar_wheel>

File: racecar_description/urdf/wheel.urdf.xacro (robot description, xacro)
@@ -1,5 +1,5 @@
 <?xml version="1.0"?>
 <robot xmlns:xacro="http://ros.org/wiki/xacro" name="racecar_wheel">
-    <xacro:macro name="racecar_wheel" params="namespace wheel_prefix parent *joint_pose">
+    <xacro:macro name="racecar_wheel" params="namespace wheel_prefix parent is_motor *joint_pose">
         <link name="${namespace}${wheel_prefix}_wheel_link">
             <inertial>
@@ -37,14 +37,16 @@
             <axis xyz="0 1 0" rpy="0 0 0" />
         </joint>
-        <transmission name="${namespace}${wheel_prefix}_wheel_trans" type="SimpleTransmission">
-            <type>transmission_interface/SimpleTransmission</type>
-            <actuator name="${namespace}${wheel_prefix}_wheel_motor">
-                <hardwareInterface>EffortJointInterface</hardwareInterface>
-                <mechanicalReduction>1</mechanicalReduction>
-            </actuator>
-            <joint name="${namespace}${wheel_prefix}_wheel">
-                <hardwareInterface>hardware_interface/EffortJointInterface</hardwareInterface>
-            </joint>
-        </transmission>
+        <xacro:if value="${is_motor}">
+            <transmission name="${namespace}${wheel_prefix}_wheel_trans" type="SimpleTransmission">
+                <type>transmission_interface/SimpleTransmission</type>
+                <actuator name="${namespace}${wheel_prefix}_wheel_motor">
+                    <hardwareInterface>EffortJointInterface</hardwareInterface>
+                    <mechanicalReduction>1</mechanicalReduction>
+                </actuator>
+                <joint name="${namespace}${wheel_prefix}_wheel">
+                    <hardwareInterface>hardware_interface/EffortJointInterface</hardwareInterface>
+                </joint>
+            </transmission>
+        </xacro:if>
     </xacro:macro>
 </robot>

Commit message: full rework of the package, C++ controller instead of python, replaced jointEffortControllers by jointVelocityControllers, fixed errors on the ackermann model and switched the car from 4WD to 2WD.

File: racecar_description/urdf/base.xacro (robot description, xacro)
@@ -24,10 +24,10 @@
                 </geometry>
             </visual>
-            <collision>
+            <!--collision>
                 <origin xyz="${ -0.03 + base_x_size/2} 0 0" rpy="0 0 0" />
                 <geometry>
                     <box size="${base_x_size} ${base_y_size*0.9} ${base_z_size}"/>
                 </geometry>
-            </collision>
+            </collision-->
         </link>
         <link name="${namespace}inertial_link">

File: racecar_description/urdf/wheel.urdf.xacro (robot description, xacro)
@@ -36,4 +36,5 @@
             <xacro:insert_block name="joint_pose"/>
             <axis xyz="0 1 0" rpy="0 0 0" />
+            <limit effort="100" velocity="400" />
         </joint>
         <xacro:if value="${is_motor}">
@@ -41,9 +42,9 @@
                 <type>transmission_interface/SimpleTransmission</type>
                 <actuator name="${namespace}${wheel_prefix}_wheel_motor">
-                    <hardwareInterface>EffortJointInterface</hardwareInterface>
+                    <hardwareInterface>hardware_interface/VelocityJointInterface</hardwareInterface>
                     <mechanicalReduction>1</mechanicalReduction>
                 </actuator>
                 <joint name="${namespace}${wheel_prefix}_wheel">
-                    <hardwareInterface>hardware_interface/EffortJointInterface</hardwareInterface>
+                    <hardwareInterface>hardware_interface/VelocityJointInterface</hardwareInterface>
                 </joint>
             </transmission>
