Commit message: swapped the continuous joints for revolute joints

File: racecar_description/urdf/hinge.urdf.xacro (robot description, xacro)
@@ -5,8 +5,8 @@
             <inertial>
                 <origin xyz="0 0 0" rpy="0 0 0" />
-                <mass value="0.100" />
-                <inertia ixx="4E-06" ixy="0"      ixz="0"
-                                     iyy="4E-06"  iyz="0"
-                                                  izz="4E-06" />
+                <mass value="1.00" />
+                <inertia ixx="0.1" ixy="0"      ixz="0"
+                                     iyy="0.1"  iyz="0"
+                                                  izz="0.1" />
             </inertial>
             <visual>
@@ -17,9 +17,10 @@
             </visual>
         </link>
-        <joint name="${namespace}${hinge_prefix}_hinge" type="continuous">
+        <joint name="${namespace}${hinge_prefix}_hinge" type="revolute">
             <parent link="${namespace}base_link"/>
             <child link="${namespace}${hinge_prefix}_hinge_link"/>
             <xacro:insert_block name="joint_pose"/>
-            <axis xyz="0 0 1" rpy="0 0 0" />
+            <axis xyz="0 0 1"/>
+            <limit upper="3.14" lower="-3.14" effort="1000.0" velocity="50.0" />
         </joint>
         <transmission name="${namespace}${hinge_prefix}_hinge_trans" type="SimpleTransmission">
