Commit message: Fixed changed the formula used to compute the inertia of the wheels

File: racecar_description/urdf/wheel.urdf.xacro (robot description, xacro)
@@ -4,14 +4,14 @@
         <link name="${namespace}${wheel_prefix}_wheel_link">
             <inertial>
-                <mass value="0.100" />
+                <mass value="0.3" />
                 <origin xyz="0 0 0" />
-                <inertia ixx="0.0002646" ixy="0"           ixz="0"
-                                         iyy="0.00041226"   iyz="0"
-                                                           izz="0.0002646" />
+                <inertia ixx="${0.3/12*(3*wheel_radius*wheel_radius + wheel_length*wheel_length)}" ixy="0"           ixz="0"
+                         iyy="${0.3/12*(3*wheel_radius*wheel_radius + wheel_length*wheel_length)}"   iyz="0"
+                         izz="${0.3/2 * wheel_radius*wheel_radius}" />
             </inertial>
             <visual>
                 <origin xyz="0 0 0" rpy="${M_PI/2} 0 0" />
                 <geometry>
-                    <mesh filename="package://racecar_description/meshes/wheel.STL" />
+                    <cylinder length="${wheel_length}" radius="${wheel_radius}" />
                 </geometry>
             </visual>
@@ -24,6 +24,6 @@
         </link>
         <gazebo reference="${namespace}${wheel_prefix}_wheel_link">
-            <mu1 value="1.0"/>
-            <mu2 value="1.0"/>
+            <mu1 value="1.5"/>
+            <mu2 value="1.5"/>
             <kp value="10000000.0" />
             <kd value="1.0" />
